Commit message: 3.0.17.20250519095033

File: DA_D03_description/urdf/DA_D03_01.urdf (robot description, URDF)
Before this commit: robot DA_D03_01, 18 links, 17 joints
Links:
- removed link neck_yaw_link
- added link head_yaw_link, mass 0.146953052787906; collision mesh filename=package://DA_D03_01_description/meshes/neck_yaw_link.STL; visual mesh filename=package://DA_D03_01_description/meshes/neck_yaw_link.STL
Joints:
- joint neck_pitch_joint: parent neck_yaw_link -> head_yaw_link
- joint neck_yaw_joint: child neck_yaw_link -> head_yaw_link
