Commit message: 1.0.0.20250731171750

File: HU_D03_description/urdf/HU_D03_03.urdf (robot description, URDF)
Before this commit: robot HU_D03_03, 40 links, 39 joints
Links:
- added link head_camera_link; visual mesh filename=package://HU_D03_description/meshes/HU_D03_03/d435.dae
- added link waist_camera_link; visual mesh filename=package://HU_D03_description/meshes/HU_D03_03/d435.dae
Joints:
- added joint head_camera_joint: type fixed, parent head_pitch_link, child head_camera_link, origin xyz=0.07453 0.0175 0.065 rpy=0.0 0.0 0.0
- added joint waist_camera_joint: type fixed, parent waist_pitch_link, child waist_camera_link, origin xyz=0.092 0.0175 0.2751 rpy=0.0 0.611 0.0

Commit message: 1.0.0.20250811102642

File: HU_D03_description/urdf/HU_D03_03.urdf (robot description, URDF)
Before this commit: robot HU_D03_03, 42 links, 41 joints
Links:
- link head_camera_link: geometry visual mesh filename=package://HU_D03_description/meshes/HU_D03_03/d435_link.STL
- link waist_camera_link: geometry visual mesh filename=package://HU_D03_description/meshes/HU_D03_03/d435_link.STL
Joints:
- joint head_camera_joint: origin xyz=0.07453 0.0175 0.065 rpy=0.0 0.0 0.0 -> xyz=0.07453 0.0175 0.065 rpy=0.0 1.5708 0.0
- joint waist_camera_joint: origin xyz=0.092 0.0175 0.2751 rpy=0.0 0.611 0.0 -> xyz=0.092 0.0175 0.2751 rpy=0.0 2.1818 0.0

Commit message: 1.0.0.20250823003145

File: HU_D03_description/urdf/HU_D03_03.urdf (robot description, URDF)
Before this commit: robot HU_D03_03, 42 links, 41 joints
Links:
- link left_ankle_roll_link: mass 1.049 -> 1.25
- link right_ankle_roll_link: mass 1.049 -> 1.25
Joints:
- joint contact_foot_tip_joint_L: origin xyz=0.144 0 -0.0625 rpy=0 0 0 -> xyz=0.154 0 -0.0625 rpy=0 0 0
- joint contact_foot_tip_joint_R: origin xyz=0.144 0 -0.0625 rpy=0 0 0 -> xyz=0.154 0 -0.0625 rpy=0 0 0

Commit message: 1.0.0.20250919221703

File: HU_D03_description/urdf/HU_D03_03.urdf (robot description, URDF)
Before this commit: robot HU_D03_03, 42 links, 41 joints
Links:
- added link left_hand_manip, mass 0.001; visual box size=0.01 0.01 0.01
- added link right_hand_manip, mass 0.001; visual box size=0.01 0.01 0.01
Joints:
- added joint left_hand_manip_joint: type fixed, parent left_hand_yaw_link, child left_hand_manip, origin xyz=0 0 0.0 rpy=0 1.5708 0
- added joint right_hand_manip_joint: type fixed, parent right_hand_yaw_link, child right_hand_manip, origin xyz=0 0 0.0 rpy=0 1.5708 0

File: HU_D04_description/urdf/HU_D04_01.urdf (robot description, URDF)
Before this commit: robot HU_D04_01, 40 links, 39 joints
Links:
- added link left_hand_manip, mass 0.001; visual box size=0.01 0.01 0.01
- added link right_hand_manip, mass 0.001; visual box size=0.01 0.01 0.01
Joints:
- added joint left_hand_manip_joint: type fixed, parent left_wrist_roll_link, child left_hand_manip, origin xyz=0 0 -0.058 rpy=0 1.5708 0
- added joint right_hand_manip_joint: type fixed, parent right_wrist_roll_link, child right_hand_manip, origin xyz=0 0 -0.058 rpy=0 1.5708 0
