Commit message: 1.0.0.20250827193641

File: HU_D04_description/urdf/HU_D04_01.urdf (robot description, URDF)
Before this commit: robot HU_D04_01, 40 links, 39 joints
Joints:
- joint left_hip_pitch_joint: origin xyz=0.017007 0.1211 0.011573 rpy=0 0 0 -> xyz=0.017007 0.1283 0.0081917 rpy=0 0 0
- joint left_hip_roll_joint: origin xyz=-0.01 0.0089101 -0.095423 rpy=0 0 0 -> xyz=-0.01 0.0016596 -0.0920417 rpy=0 0 0
- joint right_hip_pitch_joint: origin xyz=0.017007 -0.1211 0.011573 rpy=0 0 0 -> xyz=0.017007 -0.1283 0.0081917 rpy=0 0 0
- joint right_hip_roll_joint: origin xyz=-0.01 -0.0089101 -0.095423 rpy=0 0 0 -> xyz=-0.01 -0.0016596 -0.0920417 rpy=0 0 0
- joint waist_yaw_joint: origin xyz=0.0070074 0 0.10215 rpy=0 0 0 -> xyz=0 0 0.10239 rpy=0 0 0

Commit message: 1.0.0.20250905121108

File: HU_D04_description/urdf/HU_D04_01.urdf (robot description, URDF)
Before this commit: robot HU_D04_01, 40 links, 39 joints
Links:
- link left_ankle_roll_link: mass 1.577814 -> 1.206425
- link left_elbow_link: mass 1.355371 -> 1.275459
- link left_wrist_pitch_link: mass 0.74264 -> 0.658602
- link left_wrist_roll_link: mass 0.302626 -> 0.581445
- link left_wrist_yaw_link: mass 0.156822 -> 0.132906
- link right_ankle_roll_link: mass 1.577814 -> 1.206425
- link right_elbow_link: mass 1.355124 -> 1.275459
- link right_wrist_pitch_link: mass 0.744082 -> 0.658602
- link right_wrist_roll_link: mass 0.302626 -> 0.581445
- link right_wrist_yaw_link: mass 0.154827 -> 0.132906
- link waist_pitch_link: mass 10.275639 -> 11.882244

Commit message: 1.0.0.20250923095453

File: HU_D04_description/urdf/HU_D04_01.urdf (robot description, URDF)
Before this commit: robot HU_D04_01, 42 links, 41 joints
Joints:
- joint left_elbow_joint: limit lower=-2.443 upper=1.187 effort=42 velocity=19.6 -> lower=-2.443 upper=1.571 effort=42 velocity=19.6
- joint right_elbow_joint: limit lower=-2.443 upper=1.187 effort=42 velocity=19.6 -> lower=-2.443 upper=1.571 effort=42 velocity=19.6
