Commit message: fix(HU_D04_01): update link inertia and add HU_D04_01_vis.xml

File: HU_D04_description/urdf/HU_D04_01.urdf (robot description, URDF)
Before this commit: robot HU_D04_01, 42 links, 41 joints
Links:
- link left_ankle_roll_link: mass 1.206425 -> 1.021
- link left_knee_link: mass 3.004275 -> 2.958367
- link right_ankle_roll_link: mass 1.206425 -> 1.021
- link right_hip_pitch_link: mass 2.253993 -> 2.255011
- link right_hip_roll_link: mass 2.121322 -> 2.121806
- link right_knee_link: mass 2.944928 -> 2.958367
- link right_shoulder_roll_link: mass 1.727406 -> 1.740745
- link right_shoulder_yaw_link: mass 0.306436 -> 0.307657

File: HU_D04_description/urdf/HU_D04_01_with_gripper.urdf (robot description, URDF)
Before this commit: robot HU_D04_01, 52 links, 51 joints
Links:
- link left_ankle_roll_link: mass 1.206425 -> 1.021
- link left_knee_link: mass 3.004275 -> 2.958367
- link right_ankle_roll_link: mass 1.206425 -> 1.021
- link right_hip_pitch_link: mass 2.253993 -> 2.255011
- link right_hip_roll_link: mass 2.121322 -> 2.121806
- link right_knee_link: mass 2.944928 -> 2.958367
- link right_shoulder_roll_link: mass 1.727406 -> 1.740745
- link right_shoulder_yaw_link: mass 0.306436 -> 0.307657

File: HU_D04_description/urdf/HU_D04_01_with_hand.urdf (robot description, URDF)
Before this commit: robot HU_D04_01, 78 links, 77 joints
Links:
- link left_ankle_roll_link: mass 1.206425 -> 1.021
- link left_knee_link: mass 3.004275 -> 2.958367
- link right_ankle_roll_link: mass 1.206425 -> 1.021
- link right_hip_pitch_link: mass 2.253993 -> 2.255011
- link right_hip_roll_link: mass 2.121322 -> 2.121806
- link right_knee_link: mass 2.944928 -> 2.958367
- link right_shoulder_roll_link: mass 1.727406 -> 1.740745
- link right_shoulder_yaw_link: mass 0.306436 -> 0.307657
