Commit message: 1.0.0.20251016214116

File: HU_D04_description/urdf/HU_D04_01_with_hand.urdf (robot description, URDF)
Before this commit: robot HU_D04_01, 76 links, 75 joints
Links:
- added link left_transition_link, mass 0.001; visual mesh filename=../meshes/HU_D04_01/hand_transition_link.STL
- added link right_transition_link, mass 0.001; visual mesh filename=../meshes/HU_D04_01/hand_transition_link.STL
Joints:
- added joint left_transition_joint: type fixed, parent left_wrist_roll_link, child left_transition_link, origin xyz=0.0 0.0 -0.062 rpy=0 0 0
- added joint right_transition_joint: type fixed, parent right_wrist_roll_link, child right_transition_link, origin xyz=0.0 0.0 -0.062 rpy=0 0 0
- joint left_index_distal_joint: type fixed -> revolute
- joint left_index_proximal_joint: type fixed -> revolute
- joint left_index_tip_joint: type fixed -> revolute
- joint left_middle_distal_joint: type fixed -> revolute
- joint left_middle_proximal_joint: type fixed -> revolute
- joint left_middle_tip_joint: type fixed -> revolute
- joint left_pinky_distal_joint: type fixed -> revolute
- joint left_pinky_proximal_joint: type fixed -> revolute
- joint left_pinky_tip_joint: type fixed -> revolute
- joint left_ring_distal_joint: type fixed -> revolute
- joint left_ring_proximal_joint: type fixed -> revolute
- joint left_ring_tip_joint: type fixed -> revolute
- joint left_thumb_distal_joint: type fixed -> revolute
- joint left_thumb_metacarpal_joint: type fixed -> revolute
- joint left_thumb_proximal_joint: type fixed -> revolute
- joint left_thumb_tip_joint: type fixed -> revolute
- joint right_index_distal_joint: type fixed -> revolute
- joint right_index_proximal_joint: type fixed -> revolute
- joint right_index_tip_joint: type fixed -> revolute
- joint right_middle_distal_joint: type fixed -> revolute
- joint right_middle_proximal_joint: type fixed -> revolute
- joint right_middle_tip_joint: type fixed -> revolute
- joint right_pinky_distal_joint: type fixed -> revolute
- joint right_pinky_proximal_joint: type fixed -> revolute
- joint right_pinky_tip_joint: type fixed -> revolute
- joint right_ring_distal_joint: type fixed -> revolute
- joint right_ring_proximal_joint: type fixed -> revolute
- joint right_ring_tip_joint: type fixed -> revolute
- joint right_thumb_distal_joint: type fixed -> revolute
- joint right_thumb_metacarpal_joint: type fixed -> revolute
- joint right_thumb_proximal_joint: type fixed -> revolute
- joint right_thumb_tip: type fixed -> revolute
