Commit message: fix(HU_D04_01): with_hand 10 fingertip joints zero-width revolute→fixed; align right-hand tip link/joint/mesh naming with left

File: HU_D04_description/urdf/HU_D04_01_with_hand.urdf (robot description, URDF)
Before this commit: robot HU_D04_01, 78 links, 77 joints
Links:
- removed link right_index_tip
- removed link right_middle_tip
- removed link right_pinky_tip
- removed link right_ring_tip
- removed link right_thumb_tip
- added link right_index_tip_link, mass 0.001; visual mesh filename=package://HU_D04_description/meshes/HU_D04_01/right_index_t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
- added link right_middle_tip_link, mass 0.001; visual mesh filename=package://HU_D04_description/meshes/HU_D04_01/right_middle_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
- added link right_pinky_tip_link, mass 0.001; visual mesh filename=package://HU_D04_description/meshes/HU_D04_01/right_pinky_t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
- added link right_ring_tip_link, mass 0.001; visual mesh filename=package://HU_D04_description/meshes/HU_D04_01/right_ring_ti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
- added link right_thumb_tip_link, mass 0.001; visual mesh filename=package://HU_D04_description/meshes/HU_D04_01/right_thumb_t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
Joints:
- removed joint right_thumb_tip
- added joint right_thumb_tip_joint: type fixed, parent right_thumb_distal_link, child right_thumb_tip_link, origin xyz=0 0.026529 -0.0017734 rpy=-0.06675 0 0
- joint left_index_tip_joint: axis 0 1 0 -> (none); limit lower=1 upper=1 effort=1 velocity=1 -> (none); type revolute -> fixed
- joint left_middle_tip_joint: axis 0 1 0 -> (none); limit lower=1 upper=1 effort=1 velocity=1 -> (none); type revolute -> fixed
- joint left_pinky_tip_joint: axis 0 1 0 -> (none); limit lower=1 upper=1 effort=1 velocity=1 -> (none); type revolute -> fixed
- joint left_ring_tip_joint: axis 0 1 0 -> (none); limit lower=1 upper=1 effort=1 velocity=1 -> (none); type revolute -> fixed
- joint left_thumb_tip_joint: axis -1 0 0 -> (none); limit lower=0 upper=0 effort=0 velocity=0 -> (none); type revolute -> fixed
- joint right_index_tip_joint: axis 0 1 0 -> (none); child right_index_tip -> right_index_tip_link; limit lower=0 upper=0 effort=0 velocity=0 -> (none); type revolute -> fixed
- joint right_middle_tip_joint: axis 0 1 0 -> (none); child right_middle_tip -> right_middle_tip_link; limit lower=0 upper=0 effort=0 velocity=0 -> (none); type revolute -> fixed
- joint right_pinky_tip_joint: axis 0 1 0 -> (none); child right_pinky_tip -> right_pinky_tip_link; limit lower=0 upper=0 effort=0 velocity=0 -> (none); type revolute -> fixed
- joint right_ring_tip_joint: axis 0 1 0 -> (none); child right_ring_tip -> right_ring_tip_link; limit lower=0 upper=0 effort=0 velocity=0 -> (none); type revolute -> fixed
